File: Receiver/LumiCom_TIA/LTC6268-10/LMH34400.kicad_sch (KiCad schematic)
At the start: 24 parts, among them J1 TEST, J2 Conn_Coaxial, J3 Vout, J4 N_EN, J5 N_ALC, J6 Conn_Coaxial, U1 XLMH34400IDRLR

Commit message: Multiple updates
SMA, Screw terminals, track widths, added some optional 0 ohm bypass resistors
Parts:
- J1, J2, J6: footprint LumiCom_TIA:RFSOLUTIONS_CON-SMA-EDGE-S -> Connector_Coaxial:SMA_Samtec_SMA-J-P-X-ST-EM1_EdgeMount
Changed lines of the file:
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@@
 			)
 		)
-		(property "Footprint" "LumiCom_TIA:RFSOLUTIONS_CON-SMA-EDGE-S"
+		(property "Footprint" "Connector_Coaxial:SMA_Samtec_SMA-J-P-X-ST-EM1_EdgeMount"
 			(at 82.55 88.9 0)
 			(effects
@@
 			)
 		)
-		(property "Footprint" "LumiCom_TIA:RFSOLUTIONS_CON-SMA-EDGE-S"
+		(property "Footprint" "Connector_Coaxial:SMA_Samtec_SMA-J-P-X-ST-EM1_EdgeMount"
 			(at 68.58 113.03 0)
 			(effects
@@
 			)
 		)
-		(property "Footprint" "LumiCom_TIA:RFSOLUTIONS_CON-SMA-EDGE-S"
+		(property "Footprint" "Connector_Coaxial:SMA_Samtec_SMA-J-P-X-ST-EM1_EdgeMount"
 			(at 223.52 105.41 0)
 			(effects
