File: Transmitter/LumiCom_Transmitter/LumiCom_Transmitter.kicad_sch (KiCad schematic)
At the start: 38 parts, among them J1 V, J2 IN_B, J3 IN_A, J4 OUT_B, J5 OUT_A, U1 OPA2675

Commit message: Multiple updates
SMA, Screw terminals, track widths, added some optional 0 ohm bypass resistors
Parts:
- J1: footprint TerminalBlock_Phoenix:TerminalBlock_Phoenix_MPT-0,5-2-2.54_1x02_P2.54mm_Horizontal -> TerminalBlock_Phoenix:TerminalBlock_Phoenix_MKDS-1,5-2_1x02_P5.00mm_Horizontal
- J2, J3, J4, J5: footprint LumiCom_Transmitter:RFSOLUTIONS_CON-SMA-EDGE-S -> Connector_Coaxial:SMA_Samtec_SMA-J-P-X-ST-EM1_EdgeMount
