File: Transmitter/LED/LED.kicad_sch (KiCad schematic)
At the start: 11 parts, among them J1 RFPC-SMA28-F, J2 RFPC-SMA28-F, J4 Vdc

Commit message: Fixed LED pcb
Parts:
- removed J4: Vdc, TerminalBlock_Phoenix:TerminalBlock_Phoenix_MKDS-1,5-2_1x02_P5.00mm_Horizontal, symbol Connector:Screw_Terminal_01x02
- added J3: Vdc, TerminalBlock_Phoenix:TerminalBlock_Phoenix_MKDS-1,5-2_1x02_P5.00mm_Horizontal, symbol Connector:Screw_Terminal_01x02
- H1, H2, H3: footprint MountingHole:MountingHole_2.7mm_M2.5 -> MountingHole:MountingHole_3.2mm_M3_DIN965
Connections:
- net GND: now also J3.1 (Pin_1)
- net at L1.2: now also J3.2 (Pin_2)
Changed lines of the file:
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@@
 			)
 		)
-		(property "Footprint" "MountingHole:MountingHole_2.7mm_M2.5"
+		(property "Footprint" "MountingHole:MountingHole_3.2mm_M3_DIN965"
 			(at 209.55 63.5 0)
 			(effects
@@
 	)
 	(symbol
+		(lib_id "Connector:Screw_Terminal_01x02")
+		(at 52.07 97.79 180)
+		(unit 1)
+		(exclude_from_sim no)
+		(in_bom yes)
+		(on_board yes)
+		(dnp no)
+		(property "Reference" "J3"
+			(at 52.07 104.14 0)
+			(effects
+				(font
+					(size 1.27 1.27)
+				)
+			)
+		)
+		(property "Value" "Vdc"
+			(at 52.07 101.6 0)
+			(effects
+				(font
+					(size 1.27 1.27)
+				)
+			)
+		)
+		(property "Footprint" "TerminalBlock_Phoenix:TerminalBlock_Phoenix_MKDS-1,5-2_1x02_P5.00mm_Horizontal"
+			(at 52.07 97.79 0)
+			(effects
+				(font
+					(size 1.27 1.27)
+				)
+				(hide yes)
+			)
+		)
+		(property "Datasheet" "~"
+			(at 52.07 97.79 0)
+			(effects
+				(font
+					(size 1.27 1.27)
+				)
+				(hide yes)
+			)
+		)
+		(property "Description" "Generic screw terminal, single row, 01x02, script generated (kicad-library-utils/schlib/autogen/connector/)"
+			(at 52.07 97.79 0)
+			(effects
+				(font
+					(size 1.27 1.27)
+				)
+				(hide yes)
+			)
+		)
+		(pin "1"
+		)
+		(pin "2"
+		)
+		(instances
+			(project "LED"
+				(path "/cde9c444-d16b-47c2-b816-c8654de79d41"
+					(reference "J3")
+					(unit 1)
+				)
+			)
+		)
+	)
+	(symbol
 		(lib_id "power:GND")
 		(at 226.06 132.08 0)
@@
 			)
 		)
-		(property "Footprint" "MountingHole:MountingHole_2.7mm_M2.5"
+		(property "Footprint" "MountingHole:MountingHole_3.2mm_M3_DIN965"
 			(at 190.5 76.2 0)
 			(effects
@@
 			)
 		)
-		(property "Footprint" "MountingHole:MountingHole_2.7mm_M2.5"
+		(property "Footprint" "MountingHole:MountingHole_3.2mm_M3_DIN965"
 			(at 190.5 63.5 0)
 			(effects
@@
 					(unit 1)
 				)
-			)
-		)
-	)
-	(symbol
-		(lib_id "Connector:Screw_Terminal_01x02")
-		(at 52.07 95.25 0)
-		(mirror y)
-		(unit 1)
-		(exclude_from_sim no)
-		(in_bom yes)
-		(on_board yes)
-		(dnp no)
-		(fields_autoplaced yes)
-		(property "Reference" "J4"
-			(at 52.07 88.9 0)
-			(effects
-				(font
-					(size 1.27 1.27)
-				)
-			)
-		)
-		(property "Value" "Vdc"
-			(at 52.07 91.44 0)
-			(effects
-				(font
-					(size 1.27 1.27)
-				)
-			)
-		)
-		(property "Footprint" "TerminalBlock_Phoenix:TerminalBlock_Phoenix_MKDS-1,5-2_1x02_P5.00mm_Horizontal"
-			(at 52.07 95.25 0)
-			(effects
-				(font
-					(size 1.27 1.27)
-				)
-				(hide yes)
-			)
-		)
-		(property "Datasheet" "~"
-			(at 52.07 95.25 0)
-			(effects
-				(font
-					(size 1.27 1.27)
-				)
-				(hide yes)
-			)
-		)
-		(property "Description" "Generic screw terminal, single row, 01x02, script generated (kicad-library-utils/schlib/autogen/connector/)"
-			(at 52.07 95.25 0)
-			(effects
-				(font
-					(size 1.27 1.27)
-				)
-				(hide yes)
-			)
-		)
-		(pin "1"
-		)
-		(pin "2"
-		)
-		(instances
-			(project "LED"
-				(path "/cde9c444-d16b-47c2-b816-c8654de79d41"
-					(reference "J4")
-					(unit 1)
-				)

Commit message: LED corrections finished
Parts:
- C1, C2: value 1uF -> .1uF; footprint Capacitor_SMD:C_0603_1608Metric_Pad1.08x0.95mm_HandSolder -> Capacitor_SMD:C_0402_1005Metric_Pad0.74x0.62mm_HandSolder; Mfr (none) -> KYOCERA AVX; Mfr number (none) -> 530L104KT16; Mouser (none) -> 581-530L104KT16
- J1, J2: Mfr (none) -> Global Connector Technology (GCT); Mfr number (none) -> RFPC-SMA28-F; Mouser (none) -> 640-RFPCSMA28F
- J3: now left out of the parts list
- L1: Mfr (none) -> Wurth Elektronik; Mfr number (none) -> 744918220; Mouser (none) -> 710-744918220
- LED1, LED2: LCSC C3646952 -> (none)

Commit message: Last fix Led pcb
Parts:
- C1, C2: Manufacturer (none) -> KYOCERA AVX; Manufacturer Part Number (none) -> 530L104KT16; Mfr KYOCERA AVX -> (none); Mfr number 530L104KT16 -> (none); Mouser 581-530L104KT16 -> (none); Mouser Part Number (none) -> 581-530L104KT16
- H1, H2, H3: value MountingHole -> M3 Mounting hole
- J1, J2: Manufacturer (none) -> Global Connector Technology (GCT); Manufacturer Part Number (none) -> RFPC-SMA28-F; Mfr Global Connector Technology (GCT) -> (none); Mfr number RFPC-SMA28-F -> (none); Mouser 640-RFPCSMA28F -> (none); Mouser Part Number (none) -> 640-RFPCSMA28F
- L1: Manufacturer (none) -> Wurth Elektronik; Manufacturer Part Number (none) -> 744918220; Mfr Wurth Elektronik -> (none); Mfr number 744918220 -> (none); Mouser 710-744918220 -> (none); Mouser Part Number (none) -> 710-744918220
Other:
- moved on the sheet: C2, J2, LED1
